Commit message: feat: 完成二轮平衡车模型调优并实现Gazebo仿真运动
- 修复 robot.xacro 中轮子关节（Left/RightWheel_Joint）的XYZ偏移问题，解决STL模型在Gazebo中嵌入底盘的问题。
- 配置 ros2_control.yaml 并集成控制器（diff_drive_controller/balancer_controller），完成底盘驱动配置。
- 完善 gazebo.launch.py，实现一键启动 gzserver、spawn_entity 及 controller_manager。
- 验证仿真环境：机器人模型正确加载

File: src/robot/urdf/robot.xacro (robot description, xacro)
@@ -2,4 +2,5 @@
 <robot xmlns:xacro="http://www.ros.org/wiki/xacro" name="robot">
 <xacro:arg name="config_path" default="$(find robot)/config/ros2_control.yaml"/>
+<xacro:arg name="mesh_path" default="$(find robot)/meshes"/>
   <!-- ======= Base Link ======= -->
   <link name="base_link">
@@ -13,5 +14,5 @@
       <origin xyz="0 0 0" rpy="0 0 0" />
       <geometry>
-        <mesh filename="package://robot/meshes/base_link.STL" />
+        <mesh filename="file://$(arg mesh_path)/base_link.STL" />
       </geometry>
       <material name="silver">
@@ -22,5 +23,5 @@
       <origin xyz="0 0 0" rpy="0 0 0" />
       <geometry>
-        <mesh filename="package://robot/meshes/base_link.STL" />
+        <mesh filename="file://$(arg mesh_path)/base_link.STL" />
       </geometry>
     </collision>
@@ -41,5 +42,5 @@
       <origin xyz="0 0 0" rpy="0 0 0" />
       <geometry>
-        <mesh filename="package://robot/meshes/LeftWheel_Link.STL" />
+        <mesh filename="file://$(arg mesh_path)/LeftWheel_Link.STL" />
       </geometry>
       <material name="black">
@@ -50,5 +51,5 @@
       <origin xyz="0 0 0" rpy="0 0 0" />
       <geometry>
-        <mesh filename="package://robot/meshes/LeftWheel_Link.STL" />
+        <mesh filename="file://$(arg mesh_path)/LeftWheel_Link.STL" />
       </geometry>
     </collision>
@@ -72,5 +73,5 @@
       <origin xyz="0 0 0" rpy="0 0 0" />
       <geometry>
-        <mesh filename="package://robot/meshes/RightWheel_Link.STL" />
+        <mesh filename="file://$(arg mesh_path)/RightWheel_Link.STL" />
       </geometry>
       <material name="black">
@@ -81,5 +82,5 @@
       <origin xyz="0 0 0" rpy="0 0 0" />
       <geometry>
-        <mesh filename="package://robot/meshes/RightWheel_Link.STL" />
+        <mesh filename="file://$(arg mesh_path)/RightWheel_Link.STL" />
       </geometry>
     </collision>
@@ -94,16 +95,16 @@
   <!-- ======= Joints ======= -->
   <joint name="LeftWheel_Joint" type="continuous">
-    <origin xyz="0.00018658 0.0385 0.009" rpy="-1.5708 0 0" />
+    <origin xyz="0.00018658 0.115 -0.020" rpy="0 0 0" />
     <parent link="base_link" />
     <child link="LeftWheel_Link" />
-    <axis xyz="0 0 1" />
+    <axis xyz="0 1 0" />
     <limit effort="10.0" velocity="5.0" />
     <dynamics damping="0.01" friction="0.01" />
   </joint>
   <joint name="RightWheel_Joint" type="continuous">
-    <origin xyz="0.00018658 -0.0385 0.009" rpy="-1.5708 0 0" />
+    <origin xyz="0.00018658 -0.115 -0.020" rpy="0 0 0" />
     <parent link="base_link" />
     <child link="RightWheel_Link" />
-    <axis xyz="0 0 1" />
+    <axis xyz="0 1 0" />
     <limit effort="10.0" velocity="5.0" />
     <dynamics damping="0.01" friction="0.01" />
